File: DAQv4-26-27.kicad_sch (KiCad schematic)
At the start: 10 parts, among them IC1 ADS7066IRTER, IC2 ADS7066IRTER, J1 Screw_Terminal_01x02, U1 STM32H745IITx, U2 AD8495

Commit message: updates to amp
Parts:
- added R1: 1M, PCM_SparkFun-Resistor:R_0402_1005Metric, symbol PCM_SparkFun-Resistor:1M_0402
Connections:
- net GND: now also R1.1
- net at C1.1, C5.2, J1.1 (Pin_1)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: now also R1.2
Other:
- moved on the sheet: J1
Changed lines of the file:
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@@
 	(paper "C")
+	(junction
+		(at 25.4 212.09)
+		(diameter 0)
+		(color 0 0 0 0)
+	)
 	(junction
 		(at 31.75 208.28)
@@
 	)
 	(junction
+		(at 25.4 207.01)
+		(diameter 0)
+		(color 0 0 0 0)
+	)
+	(junction
 		(at 71.12 205.74)
 		(diameter 0)
@@
 	(wire
 		(pts
+			(xy 25.4 212.09) (xy 25.4 213.36)
+		)
+		(stroke
+			(width 0)
+			(type default)
+		)
+	)
+	(wire
+		(pts
 			(xy 49.53 191.77) (xy 57.15 191.77)
 		)
@@
 	(wire
 		(pts
+			(xy 25.4 207.01) (xy 25.4 212.09)
+		)
+		(stroke
+			(width 0)
+			(type default)
+		)
+	)
+	(wire
+		(pts
+			(xy 24.13 207.01) (xy 25.4 207.01)
+		)
+		(stroke
+			(width 0)
+			(type default)
+		)
+	)
+	(wire
+		(pts
+			(xy 25.4 207.01) (xy 29.21 207.01)
+		)
+		(stroke
+			(width 0)
+			(type default)
+		)
+	)
+	(wire
+		(pts
 			(xy 52.07 213.36) (xy 52.07 222.25)
 		)
@@
 		(pts
 			(xy 71.12 205.74) (xy 78.74 205.74)
+		)
+		(stroke
+			(width 0)
+			(type default)
+		)
+	)
+	(wire
+		(pts
+			(xy 24.13 204.47) (xy 29.21 204.47)
 		)
 		(stroke
@@
 	)
 	(symbol
+		(lib_id "PCM_SparkFun-Resistor:1M_0402")
+		(at 25.4 214.63 90)
+		(unit 1)
+		(body_style 1)
+		(exclude_from_sim no)
+		(in_bom yes)
+		(on_board yes)
+		(in_pos_files yes)
+		(dnp no)
+		(property "Reference" "R1"
+			(at 27.94 213.3599 90)
+			(show_name no)
+			(do_not_autoplace no)
+			(effects
+				(font
+					(size 1.27 1.27)
+				)
+				(justify right)
+			)
+		)
+		(property "Value" "1M"
+			(at 27.94 215.8999 90)
+			(show_name no)
+			(do_not_autoplace no)
+			(effects
+				(font
+					(size 1.27 1.27)
+				)
+				(justify right)
+			)
+		)
+		(property "Footprint" "PCM_SparkFun-Resistor:R_0402_1005Metric"
+			(at 29.972 214.63 0)
+			(hide yes)
+			(show_name no)
+			(do_not_autoplace no)
+			(effects
+				(font
+					(size 1.27 1.27)
+				)
+			)
+		)
+		(property "Datasheet" "https://www.vishay.com/docs/20035/dcrcwe3.pdf"
+			(at 34.29 215.9 0)
+			(hide yes)
+			(show_name no)
+			(do_not_autoplace no)
+			(effects
+				(font
+					(size 1.27 1.27)
+				)
+			)
+		)
+		(property "Description" "Resistor"
+			(at 36.83 214.63 0)
+			(hide yes)
+			(show_name no)
+			(do_not_autoplace no)
+			(effects
+				(font
+					(size 1.27 1.27)
+				)
+			)
+		)
+		(property "PROD_ID" "RES-15185"
+			(at 32.258 214.63 0)
+			(hide yes)
+			(show_name no)
+			(do_not_autoplace no)
+			(effects
+				(font
+					(size 1.27 1.27)
+				)
+			)
+		)
+		(pin "1"
+		)
+		(pin "2"
+		)
+		(instances
+			(project "DAQv4-26-27"
+				(path "/cbe418a7-f727-405b-87dd-9a1de7bc4b30"
+					(reference "R1")
+					(unit 1)
+				)
+			)
+		)
+	)
+	(symbol
+		(lib_id "power:GND")
+		(at 25.4 217.17 0)
+		(unit 1)
+		(body_style 1)
+		(exclude_from_sim no)
+		(in_bom yes)
+		(on_board yes)
+		(in_pos_files yes)
+		(dnp no)
+		(fields_autoplaced yes)
+		(property "Reference" "#PWR08"
+			(at 25.4 223.52 0)
+			(hide yes)
+			(show_name no)
+			(do_not_autoplace no)
+			(effects
+				(font
+					(size 1.27 1.27)
+				)
+			)
+		)
+		(property "Value" "GND"
+			(at 25.4 222.25 0)
+			(show_name no)
+			(do_not_autoplace no)
+			(effects
+				(font
+					(size 1.27 1.27)
+				)
+			)
+		)
+		(property "Footprint" ""
+			(at 25.4 217.17 0)
+			(hide yes)
+			(show_name no)
+			(do_not_autoplace no)
+			(effects
+				(font
+					(size 1.27 1.27)
+				)
+			)
+		)
+		(property "Datasheet" ""
+			(at 25.4 217.17 0)
+			(hide yes)
+			(show_name no)
+			(do_not_autoplace no)
+			(effects
+				(font
+					(size 1.27 1.27)
+				)
+			)
+		)
+		(property "Description" "Power symbol creates a global label with name \"GND\" , ground"
+			(at 25.4 217.17 0)
+			(hide yes)
+			(show_name no)
+			(do_not_autoplace no)
+			(effects
+				(font
+					(size 1.27 1.27)
+				)
+			)
+		)
+		(pin "1"
+		)
+		(instances
+			(project "DAQv4-26-27"
+				(path "/cbe418a7-f727-405b-87dd-9a1de7bc4b30"
+					(reference "#PWR08")
+					(unit 1)
+				)
+			)
+		)
+	)
+	(symbol
 		(lib_id "power:GND")
 		(at 31.75 189.23 180)
@@
 	(symbol
 		(lib_id "Connector:Screw_Terminal_01x02")
-		(at 24.13 207.01 180)
+		(at 19.05 207.01 180)
 		(unit 1)
 		(body_style 1)
@@
 		(fields_autoplaced yes)
 		(property "Reference" "J1"
-			(at 24.13 198.12 0)
+			(at 19.05 198.12 0)
 			(show_name no)
 			(do_not_autoplace no)
@@
 		)
 		(property "Value" "Screw_Terminal_01x02"
-			(at 24.13 200.66 0)
+			(at 19.05 200.66 0)
 			(show_name no)
 			(do_not_autoplace no)
@@
 		)
 		(property "Footprint" ""
-			(at 24.13 207.01 0)
+			(at 19.05 207.01 0)
 			(hide yes)
 			(show_name no)
@@
 		)
 		(property "Datasheet" ""
-			(at 24.13 207.01 0)
+			(at 19.05 207.01 0)
 			(hide yes)
 			(show_name no)
@@
 		)
 		(property "Description" "Generic screw terminal, single row, 01x02, script generated (kicad-library-utils/schlib/autogen/connector/)"
-			(at 24.13 207.01 0)
+			(at 19.05 207.01 0)
 			(hide yes)
 			(show_name no)
@@
 	)
 	(group "Thermocouple term+amp"
-		(members "2595228c-fb70-4637-8086-07af2e9cad79" "88204cb2-88ff-49df-a35f-e85755364738"
-			"98502d35-e765-4d55-8412-bafec1831bdc" "b409200e-d020-40ca-9fa3-e572bc93dbbd"
+		(members "17021c25-3c31-4c21-83bd-e797f0296c43" "2595228c-fb70-4637-8086-07af2e9cad79"
+			"5f6adae9-c578-479e-8b7f-7ef349f9124b" "617ccc6b-009d-4911-b16f-24b4b7d23d3f"
+			"6314cb00-d6c1-4063-9400-9623f2361659" "6bfe13c0-2cb3-47cf-ab4f-43fb908fb084"
+			"88204cb2-88ff-49df-a35f-e85755364738" "98502d35-e765-4d55-8412-bafec1831bdc"
+			"af4ef2c0-c9d8-4d8a-b7b0-b61e150eb881" "b409200e-d020-40ca-9fa3-e572bc93dbbd"
 			"cbbf37d6-0fe6-469e-a36e-b484304837de" "df93a123-db0a-4efc-8e75-17395aa494fb"
 		)
